File: CAN.kicad_sch (KiCad schematic)
At the start: 9 parts, among them J6 Conn_01x08, U4 ISO1050DUB

Commit message: Done with first pass, switching current amp due to stocking issues
Parts:
- C1: MPN (none) -> C57112
- C12: MPN (none) -> C14663
- R: MPN (none) -> C23182
- U4: LCSC (none) -> C16428; MPN (none) -> C16428
Changed lines of the file:
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@@
+      (effects (font (size 1.27 1.27)) hide)
+    )
+    (property "MPN" "C23182" (at 114.935 107.95 0)
       (effects (font (size 1.27 1.27)) hide)
     )
@@
       (effects (font (size 1.27 1.27)) hide)
     )
+    (property "MPN" "C14663" (at 160.02 105.41 0)
+      (effects (font (size 1.27 1.27)) hide)
+    )
     (pin "1")
     (pin "2")
@@
       (effects (font (size 1.27 1.27)) hide)
     )
+    (property "MPN" "C57112" (at 137.16 109.22 0)
+      (effects (font (size 1.27 1.27)) hide)
+    )
     (pin "1")
     (pin "2")
@@
     )
     (property "Datasheet" "http://www.ti.com/lit/ds/symlink/iso1050.pdf" (at 90.805 102.235 0)
+      (effects (font (size 1.27 1.27)) hide)
+    )
+    (property "LCSC" "C16428" (at 90.805 100.965 0)
+      (effects (font (size 1.27 1.27)) hide)
+    )
+    (property "MPN" "C16428" (at 90.805 100.965 0)
       (effects (font (size 1.27 1.27)) hide)
     )
@@
       (effects (font (size 1.27 1.27)) hide)
     )
+    (property "MPN" "C23182" (at 114.935 99.06 0)
+      (effects (font (size 1.27 1.27)) hide)
+    )
     (pin "1")
     (pin "2")
@@
       (effects (font (size 1.27 1.27)) hide)
     )
+    (property "MPN" "C14663" (at 55.88 101.6 0)
+      (effects (font (size 1.27 1.27)) hide)
+    )
