File: DC INPUT.kicad_sch (KiCad schematic)
At the start: 17 parts, among them J3 Screw_Terminal_01x01, Q3 HYG017N10NS1TA, U17 LM5060

Commit message: Done with first pass, switching current amp due to stocking issues
Parts:
- C1: MPN (none) -> C2843466
- C1: MPN (none) -> C28233
- Q3: MPN (none) -> C5205219
- R11: MPN (none) -> C149504
- R11: MPN (none) -> C865510
- R11: MPN (none) -> C5159707
- R11: MPN (none) -> C351568
- U17: MPN (none) -> C2676940
Changed lines of the file:
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@@
+      (effects (font (size 1.27 1.27)) hide)
+    )
+    (property "MPN" "C5205219" (at 111.125 81.28 0)
       (effects (font (size 1.27 1.27)) hide)
     )
@@
     )
     (property "LCSC" "C149504" (at 80.645 91.44 0)
+      (effects (font (size 1.27 1.27)) hide)
+    )
+    (property "MPN" "C149504" (at 80.645 91.44 0)
       (effects (font (size 1.27 1.27)) hide)
     )
@@
       (effects (font (size 1.27 1.27)) hide)
     )
+    (property "MPN" "C2843466" (at 45.085 83.82 0)
+      (effects (font (size 1.27 1.27)) hide)
+    )
     (pin "1")
     (pin "2")
@@
       (effects (font (size 1.27 1.27)) hide)
     )
+    (property "MPN" "C865510" (at 80.645 100.33 0)
+      (effects (font (size 1.27 1.27)) hide)
+    )
     (pin "1")
     (pin "2")
@@
       (effects (font (size 1.27 1.27)) hide)
     )
+    (property "MPN" "C5159707" (at 102.87 83.82 0)
+      (effects (font (size 1.27 1.27)) hide)
+    )
     (pin "1")
     (pin "2")
@@
     )
     (property "LCSC" "C5159707" (at 105.41 83.82 0)
+      (effects (font (size 1.27 1.27)) hide)
+    )
+    (property "MPN" "C5159707" (at 105.41 83.82 0)
       (effects (font (size 1.27 1.27)) hide)
     )
@@
       (effects (font (size 1.27 1.27)) hide)
     )
+    (property "MPN" "C28233" (at 133.35 110.49 0)
+      (effects (font (size 1.27 1.27)) hide)
+    )
     (pin "1")
     (pin "2")
@@
     )
     (property "LCSC" "C2676940" (at 108.585 100.965 0)
+      (effects (font (size 1.27 1.27)) hide)
+    )
+    (property "MPN" "C2676940" (at 108.585 100.965 0)
       (effects (font (size 1.27 1.27)) hide)
     )
@@
       (effects (font (size 1.27 1.27)) hide)
     )
+    (property "MPN" "C351568" (at 80.645 109.22 0)
+      (effects (font (size 1.27 1.27)) hide)
+    )
