File: MCU.kicad_sch (KiCad schematic)
At the start: 22 parts, among them J9 Conn_02x07_Odd_Even, SW1 SW_DIP_x01, SW2 SW_DIP_x01, U1 STM32G431CBUx, U2 DNP LM4040DBZ-2.5

Commit message: Done with first pass, switching current amp due to stocking issues
Parts:
- C1: MPN (none) -> C28233
- D2: MPN (none) -> C2297
- D3: MPN (none) -> C2296
- D4: MPN (none) -> C84256
- FB1: MPN (none) -> C1002
- J9: MPN (none) -> C2881912
- R1, R2: MPN (none) -> C25197
- R3: MPN (none) -> C22775
- SW1, SW2: MPN (none) -> C318884
- U1: MPN (none) -> C529356
Changed lines of the file:
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@@
+      (effects (font (size 1.27 1.27)) hide)
+    )
+    (property "MPN" "C25197" (at 43.815 149.225 0)
       (effects (font (size 1.27 1.27)) hide)
     )
@@
       (effects (font (size 1.27 1.27)) hide)
     )
+    (property "MPN" "C318884" (at 68.58 155.575 0)
+      (effects (font (size 1.27 1.27)) hide)
+    )
     (pin "1")
     (pin "2")
@@
     )
     (property "LCSC" "C28233" (at 173.99 60.325 0)
+      (effects (font (size 1.27 1.27)) hide)
+    )
+    (property "MPN" "C28233" (at 173.99 60.325 0)
       (effects (font (size 1.27 1.27)) hide)
     )
@@
       (effects (font (size 1.27 1.27)) hide)
     )
+    (property "MPN" "C22775" (at 107.315 22.86 0)
+      (effects (font (size 1.27 1.27)) hide)
+    )
     (pin "1")
     (pin "2")
@@
     )
     (property "LCSC" "C28233" (at 50.8 50.8 0)
+      (effects (font (size 1.27 1.27)) hide)
+    )
+    (property "MPN" "C28233" (at 50.8 50.8 0)
       (effects (font (size 1.27 1.27)) hide)
     )
@@
       (effects (font (size 1.27 1.27)) hide)
     )
+    (property "MPN" "C28233" (at 57.15 161.925 0)
+      (effects (font (size 1.27 1.27)) hide)
+    )
     (pin "1")
     (pin "2")
@@
       (effects (font (size 1.27 1.27)) hide)
     )
+    (property "MPN" "C2296" (at 107.315 31.75 0)
+      (effects (font (size 1.27 1.27)) hide)
+    )
     (pin "1")
     (pin "2")
@@
     )
     (property "LCSC" "C28233" (at 53.34 86.995 0)
+      (effects (font (size 1.27 1.27)) hide)
+    )
+    (property "MPN" "C28233" (at 53.34 86.995 0)
       (effects (font (size 1.27 1.27)) hide)
     )
@@
       (effects (font (size 1.27 1.27)) hide)
     )
+    (property "MPN" "C25197" (at 34.925 121.285 0)
+      (effects (font (size 1.27 1.27)) hide)
+    )
     (pin "1")
     (pin "2")
@@
       (effects (font (size 1.27 1.27)) hide)
     )
+    (property "MPN" "C22775" (at 127.635 22.86 0)
+      (effects (font (size 1.27 1.27)) hide)
+    )
     (pin "1")
     (pin "2")
@@
       (effects (font (size 1.27 1.27)) hide)
     )
+    (property "MPN" "C2297" (at 127.635 31.75 0)
+      (effects (font (size 1.27 1.27)) hide)
+    )
     (pin "1")
     (pin "2")
@@
     )
     (property "LCSC" "C1002" (at 139.065 48.895 0)
+      (effects (font (size 1.27 1.27)) hide)
+    )
+    (property "MPN" "C1002" (at 139.065 48.895 0)
       (effects (font (size 1.27 1.27)) hide)
     )
@@
     )
     (property "LCSC" "C529356" (at 131.445 103.505 0)
+      (effects (font (size 1.27 1.27)) hide)
+    )
+    (property "MPN" "C529356" (at 131.445 103.505 0)
       (effects (font (size 1.27 1.27)) hide)
     )
@@
       (effects (font (size 1.27 1.27)) hide)
     )
+    (property "MPN" "C28233" (at 19.05 50.8 0)
+      (effects (font (size 1.27 1.27)) hide)
+    )
     (pin "1")
     (pin "2")
@@
       (effects (font (size 1.27 1.27)) hide)
     )
+    (property "MPN" "C84256" (at 86.995 31.75 0)
+      (effects (font (size 1.27 1.27)) hide)
+    )
     (pin "1")
     (pin "2")
@@
     )
     (property "LCSC" "C318884" (at 44.45 114.935 0)
+      (effects (font (size 1.27 1.27)) hide)
+    )
+    (property "MPN" "C318884" (at 44.45 114.935 0)
       (effects (font (size 1.27 1.27)) hide)
     )
@@
     )
     (property "LCSC" "C2881912" (at 191.135 129.54 0)
+      (effects (font (size 1.27 1.27)) hide)
+    )
+    (property "MPN" "C2881912" (at 191.135 129.54 0)
       (effects (font (size 1.27 1.27)) hide)
     )
@@
       (effects (font (size 1.27 1.27)) hide)
     )
+    (property "MPN" "C28233" (at 19.05 24.765 0)
+      (effects (font (size 1.27 1.27)) hide)
+    )
     (pin "1")
     (pin "2")
@@
       (effects (font (size 1.27 1.27)) hide)
     )
+    (property "MPN" "C28233" (at 50.8 24.765 0)
+      (effects (font (size 1.27 1.27)) hide)
+    )
     (pin "1")
     (pin "2")
@@
       (effects (font (size 1.27 1.27)) hide)
     )
+    (property "MPN" "C22775" (at 86.995 22.86 0)
+      (effects (font (size 1.27 1.27)) hide)
+    )
