File: SPI.kicad_sch (KiCad schematic)
At the start: 6 parts, among them J1 47272-0001, U5 SN65LVDS31D, U6 SN65LVDS33D

Commit message: Done with first pass, switching current amp due to stocking issues
Parts:
- C12, C13: MPN (none) -> C14663
- J1: MPN (none) -> C711350
- R7: MPN (none) -> C22775
- U5: MPN (none) -> C1508988
- U6: LCSC (none) -> C1508989
Changed lines of the file:
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@@
+      (effects (font (size 1.27 1.27)) hide)
+    )
+    (property "MPN" "C14663" (at 161.29 70.485 0)
       (effects (font (size 1.27 1.27)) hide)
     )
@@
     )
     (property "LCSC" "C1508988" (at 119.38 73.025 0)
+      (effects (font (size 1.27 1.27)) hide)
+    )
+    (property "MPN" "C1508988" (at 119.38 73.025 0)
       (effects (font (size 1.27 1.27)) hide)
     )
@@
       (effects (font (size 1.27 1.27)) hide)
     )
+    (property "MPN" "C14663" (at 157.48 128.905 0)
+      (effects (font (size 1.27 1.27)) hide)
+    )
     (pin "1")
     (pin "2")
@@
     )
     (property "LCSC" "C711350" (at 205.74 93.345 0)
+      (effects (font (size 1.27 1.27)) hide)
+    )
+    (property "MPN" "C711350" (at 205.74 93.345 0)
       (effects (font (size 1.27 1.27)) hide)
     )
@@
       (effects (font (size 1.27 1.27)) hide)
     )
+    (property "MPN" "C22775" (at 63.5 133.985 0)
+      (effects (font (size 1.27 1.27)) hide)
+    )
     (pin "1")
     (pin "2")
@@
       (effects (font (size 1.27 1.27)) hide)
     )
+    (property "LCSC" "C1508989" (at 119.38 131.445 0)
+      (effects (font (size 1.27 1.27)) hide)
+    )
